File: Drone_ESC_2lag/STSPIN32G4.kicad_sch (KiCad schematic)
At the start: 21 parts, among them IC1 STSPIN32G4, SW1 JS102011SAQN, Y1 24.000MHz

Commit message: Næsten færdig med PCB, retter fejl
Parts:
- removed SW1: JS102011SAQN, Switch:SW_JS102011SAQN, symbol Switch:SW_Nidec_CAS-120A1
- added C19: 100nF, Capacitor_SMD:C_0805_2012Metric_Pad1.18x1.45mm_HandSolder, symbol Device:C
Connections:
- net GND: now also C19.1
- net at R1.1: now also IC1.59 (PB8), C19.2
- net PA15: no longer names the net of IC1.51 (PA15)
- net PB3: no longer names the net of IC1.54 (PB3)
- net PC4: no longer names the net of IC1.21 (PC4)
- net USB_D+: no longer names the net of IC1.48 (PA12)
- net USB_D-: no longer names the net of IC1.47 (PA11)
- no-connect marks 17 -> 22
Other:
- note removed: "JTDI SWCLK / JTCK SWDIO / JTMS"
- note removed: "SWO / JTDO"
- moved on the sheet: R1
